File: electronics/tongueboard/tongueboard.brd (EAGLE design)
At the start: 29 x 69 mm, 258 parts

Commit message: tongueboard ready for release.
Other:
- outline, holes or cut-outs redrawn
Changed lines of the file:
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@@
 <setting verticaltext="up"/>
 </settings>
-<grid distance="9.84251969" unitdist="mil" unit="mil" style="lines" multiple="1" display="yes" altdistance="0.025" altunitdist="inch" altunit="inch"/>
+<grid distance="0.25" unitdist="mm" unit="mm" style="lines" multiple="1" display="yes" altdistance="0.025" altunitdist="inch" altunit="inch"/>
 <layers>
 <layer number="1" name="Top" color="4" fill="1" visible="yes" active="yes"/>
@@
 <board>
 <plain>
-<wire x1="6.25" y1="33.5" x2="0" y2="27.25" width="0.2" layer="20"/>
-<wire x1="0" y1="27.25" x2="0" y2="0" width="0.2" layer="20"/>
-<wire x1="22.75" y1="33.5" x2="29" y2="27.25" width="0.2" layer="20"/>
-<wire x1="29" y1="27.25" x2="29" y2="0" width="0.2" layer="20"/>
-<wire x1="6.25" y1="33.5" x2="6.25" y2="69" width="0.2" layer="20"/>
-<wire x1="6.25" y1="69" x2="22.75" y2="69" width="0.2" layer="20"/>
-<wire x1="22.75" y1="69" x2="22.75" y2="33.5" width="0.2" layer="20"/>
-<wire x1="0" y1="0" x2="29" y2="0" width="0.2" layer="20"/>
+<wire x1="0.32218125" y1="27.57218125" x2="5.92781875" y2="33.17781875" width="0.2" layer="20"/>
+<wire x1="5.92781875" y1="33.17781875" x2="6.25" y2="33.955634375" width="0.2" layer="20" curve="44.999837"/>
+<wire x1="6.25" y1="33.955634375" x2="6.25" y2="68.7" width="0.2" layer="20"/>
+<wire x1="6.25" y1="68.7" x2="6.55" y2="69" width="0.2" layer="20" curve="-90"/>
+<wire x1="6.55" y1="69" x2="22.45" y2="69" width="0.2" layer="20"/>
+<wire x1="22.45" y1="69" x2="22.75" y2="68.7" width="0.2" layer="20" curve="-90"/>
+<wire x1="22.75" y1="68.7" x2="22.75" y2="33.955634375" width="0.2" layer="20"/>
+<wire x1="0.32218125" y1="27.57218125" x2="0" y2="26.794365625" width="0.2" layer="20" curve="44.999837"/>
+<wire x1="0" y1="26.794365625" x2="0" y2="1.1" width="0.2" layer="20"/>
+<wire x1="0" y1="1.1" x2="1.1" y2="0" width="0.2" layer="20" curve="90"/>
+<wire x1="1.1" y1="0" x2="27.9" y2="0" width="0.2" layer="20"/>
+<wire x1="22.75" y1="33.955634375" x2="23.07218125" y2="33.17781875" width="0.2" layer="20" curve="44.999885"/>
+<wire x1="23.07218125" y1="33.17781875" x2="28.67781875" y2="27.57218125" width="0.2" layer="20"/>
+<wire x1="28.67781875" y1="27.57218125" x2="29" y2="26.794365625" width="0.2" layer="20" curve="-44.999837"/>
+<wire x1="27.9" y1="0" x2="29" y2="1.1" width="0.2" layer="20" curve="90"/>
+<wire x1="29" y1="1.1" x2="29" y2="26.794365625" width="0.2" layer="20"/>
 <text x="22.1993" y="60.5718" size="2.54" layer="16" font="vector" rot="MR0">Mouth.IO</text>
 <text x="23.8157" y="28.6218" size="0.8128" layer="16" font="vector" rot="MR0">Copyright 2013 Zach Hoeken</text>
@@
 <text x="0.612" y="4.4624" size="0.6096" layer="21">C14</text>
 <text x="0.612" y="2.913" size="0.6096" layer="21">C15</text>
-<text x="2.1868" y="27.043" size="0.6096" layer="21">A0</text>
-<text x="3.7362" y="27.043" size="0.6096" layer="21">A1</text>
-<text x="5.2856" y="27.043" size="0.6096" layer="21">A2</text>
-<text x="6.835" y="27.043" size="0.6096" layer="21">A3</text>
-<text x="8.3844" y="27.043" size="0.6096" layer="21">A4</text>
-<text x="9.9338" y="27.043" size="0.6096" layer="21">A5</text>
-<text x="11.4832" y="27.043" size="0.6096" layer="21">A6</text>
-<text x="13.0326" y="27.043" size="0.6096" layer="21">A7</text>
-<text x="14.582" y="27.043" size="0.6096" layer="21">A8</text>
-<text x="16.1314" y="27.043" size="0.6096" layer="21">A9</text>
-<text x="17.6808" y="27.043" size="0.6096" layer="21">A10</text>
-<text x="19.2302" y="27.043" size="0.6096" layer="21">A11</text>
-<text x="20.7796" y="27.043" size="0.6096" layer="21">A12</text>
-<text x="22.329" y="27.043" size="0.6096" layer="21">A13</text>
-<text x="23.8784" y="27.043" size="0.6096" layer="21">A14</text>
-<text x="25.4278" y="27.043" size="0.6096" layer="21">A15</text>
+<text x="2.6868" y="1.043" size="0.6096" layer="21">A0</text>
+<text x="4.2362" y="1.043" size="0.6096" layer="21">A1</text>
+<text x="5.7856" y="1.043" size="0.6096" layer="21">A2</text>
+<text x="7.335" y="1.043" size="0.6096" layer="21">A3</text>
+<text x="8.8844" y="1.043" size="0.6096" layer="21">A4</text>
+<text x="10.4338" y="1.043" size="0.6096" layer="21">A5</text>
+<text x="11.9832" y="1.043" size="0.6096" layer="21">A6</text>
+<text x="13.5326" y="1.043" size="0.6096" layer="21">A7</text>
+<text x="15.082" y="1.043" size="0.6096" layer="21">A8</text>
+<text x="16.6314" y="1.043" size="0.6096" layer="21">A9</text>
+<text x="18.1808" y="1.043" size="0.6096" layer="21">A10</text>
+<text x="19.7302" y="1.043" size="0.6096" layer="21">A11</text>
+<text x="21.2796" y="1.043" size="0.6096" layer="21">A12</text>
+<text x="22.829" y="1.043" size="0.6096" layer="21">A13</text>
+<text x="24.3784" y="1.043" size="0.6096" layer="21">A14</text>
+<text x="25.9278" y="1.043" size="0.6096" layer="21">A15</text>
 <text x="20.1057" y="51.4868" size="1.27" layer="16" font="vector" rot="MR0">INTO MOUTH</text>
 <text x="21.47" y="31.865" size="0.8128" layer="16" font="vector" rot="MR0">mouth.io/tongueboard</text>

Commit message: routed a bunch of the brainboard.
Parts:
- U$257: device Hoektronics:FPC-PCB-32 -> Hoektronics:FPC-32-WIRE
Changed lines of the file:
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@@
 <element name="U$256" library="Hoeken" package="61MIL" value="ELECTRODE60MIL" x="26.5708" y="25.7603" rot="MR0"/>
 <element name="LOGO1" library="ohw-logo" package="OSHW_10X500_NOTEXT_COPPER" value="OSHW_LOGO_10MIL" x="7.47" y="35.6"/>
-<element name="U$257" library="Hoektronics" package="FPC-PCB-32" value="FPC-0.5-32" x="14.5" y="67.25"/>
+<element name="U$257" library="Hoektronics" package="FPC-32-WIRE" value="FPC-0.5-32" x="14.5" y="67.25"/>
 </elements>
 <signals>
