File: electronics/tongueboard/tongueboard.sch (EAGLE design)
At the start: 258 parts

Commit message: tongueboard ready for release.
Other:
- note added: "ANODE = EVEN PINS"
- note added: "CATHODE = ODD PINS"
- note added: "License: GPLv3 / Copyright 2013"
- note removed: "ANODE"
- note removed: "CATHODE"
- note removed: "License: GPLv3 / Copyright 2012"
